File: HSMC-GPIO-kicad.sch (KiCad schematic (older format))
At the start: 12 parts, among them J1 HSMC, J3 Conn_01x03_Male, J4 I2C, J5 Screw_Terminal_01x04, U2 MC78M05_TO252, U3 TCA9517

Commit message: Reroute ribbon connector protection circuitry, switch to single ribbon cable configuration.
Connections:
- net labels added: GPIO-B36, GPIO-B37, GPIO-B38, GPIO-B39, GPIO-B40, GPIO1, GPIO10, GPIO11, GPIO12, GPIO13, GPIO14, GPIO15, GPIO16, GPIO17, GPIO18, GPIO19, GPIO2, GPIO20, GPIO21, GPIO22, GPIO23, GPIO24, GPIO25, GPIO26, GPIO27, GPIO28, GPIO29, GPIO3, GPIO30, GPIO31, GPIO32, GPIO33, GPIO34, GPIO35, GPIO36, GPIO37, GPIO38, GPIO39, GPIO4, GPIO40, GPIO5, GPIO6, GPIO7, GPIO8, GPIO9
- net labels removed: GPIO-B0
- wire segments 298 -> 279
- no-connect marks 47 -> 43

Commit message: Change pin/bus labels in schematic
Connections:
- net labels added: GPIO0, GPIO[0..39]
- net labels removed: GPIO-B1, GPIO-B10, GPIO-B11, GPIO-B12, GPIO-B13, GPIO-B14, GPIO-B15, GPIO-B16, GPIO-B17, GPIO-B18, GPIO-B19, GPIO-B2, GPIO-B20, GPIO-B21, GPIO-B22, GPIO-B23, GPIO-B24, GPIO-B25, GPIO-B26, GPIO-B27, GPIO-B28, GPIO-B29, GPIO-B3, GPIO-B30, GPIO-B31, GPIO-B32, GPIO-B33, GPIO-B34, GPIO-B35, GPIO-B36, GPIO-B37, GPIO-B38, GPIO-B39, GPIO-B4, GPIO-B40, GPIO-B5, GPIO-B6, GPIO-B7, GPIO-B8, GPIO-B9, GPIO40
- wire segments 279 -> 230

Commit message: Begin routing ribbon cable connector
Parts:
- renumbered J3 to J2, J4 to J3, J5 to J4, U2 to U1, U3 to U2
Connections:
- net labels removed: GPIO-A0, GPIO-A1, GPIO-A10, GPIO-A11, GPIO-A12, GPIO-A13, GPIO-A14, GPIO-A15, GPIO-A16, GPIO-A17, GPIO-A18, GPIO-A19, GPIO-A2, GPIO-A20, GPIO-A21, GPIO-A22, GPIO-A23, GPIO-A24, GPIO-A25, GPIO-A26, GPIO-A27, GPIO-A28, GPIO-A29, GPIO-A3, GPIO-A30, GPIO-A31, GPIO-A32, GPIO-A33, GPIO-A34, GPIO-A35, GPIO-A4, GPIO-A5, GPIO-A6, GPIO-A7, GPIO-A8, GPIO-A9
- wire segments 230 -> 194
- no-connect marks 43 -> 79

Commit message: Finish initial placement and routing
Parts:
- removed C1: 100n, Capacitor_SMD:C_0805_2012Metric, symbol Device:C
- added C18, C19, C20: 10u, Capacitor_Tantalum_SMD:CP_EIA-3528-15_AVX-H, symbol Device:CP1
- added MH1, MH2: MountingHole, HSMC:MountingHole, symbol Mechanical:MountingHole
- C2, C3: footprint Capacitor_SMD:C_1210_3225Metric_Pad1.42x2.65mm_HandSolder -> Capacitor_Tantalum_SMD:CP_EIA-3528-15_AVX-H
- J4: footprint Phoenix_MFKDS:Phoenix_MFKDS-5.08_1x04_P5.08mm -> TerminalBlock:TerminalBlock_bornier-4_P5.08mm
Connections:
- wire segments 194 -> 193
Changed lines of the file:
@@
 L power:+12V #PWR019
 U 1 1 5C07431E
-P 10300 8200
-F 0 "#PWR019" H 10300 8050 50  0001 C CNN
-F 1 "+12V" H 10315 8373 50  0000 C CNN
-F 2 "" H 10300 8200 50  0001 C CNN
-F 3 "" H 10300 8200 50  0001 C CNN
-	1    10300 8200
+P 10050 8200
+F 0 "#PWR019" H 10050 8050 50  0001 C CNN
+F 1 "+12V" H 10065 8373 50  0000 C CNN
+F 2 "" H 10050 8200 50  0001 C CNN
+F 3 "" H 10050 8200 50  0001 C CNN
+	1    10050 8200
 	1    0    0    -1
 $EndComp
@@
 L power:+3V3 #PWR017
 U 1 1 5C07438E
-P 9900 8200
-F 0 "#PWR017" H 9900 8050 50  0001 C CNN
-F 1 "+3V3" H 9915 8373 50  0000 C CNN
-F 2 "" H 9900 8200 50  0001 C CNN
-F 3 "" H 9900 8200 50  0001 C CNN
-	1    9900 8200
+P 9250 8200
+F 0 "#PWR017" H 9250 8050 50  0001 C CNN
+F 1 "+3V3" H 9265 8373 50  0000 C CNN
+F 2 "" H 9250 8200 50  0001 C CNN
+F 3 "" H 9250 8200 50  0001 C CNN
+	1    9250 8200
 	1    0    0    -1
 $EndComp
@@
 L power:+5V #PWR018
 U 1 1 5C074402
-P 10100 8200
-F 0 "#PWR018" H 10100 8050 50  0001 C CNN
-F 1 "+5V" H 10115 8373 50  0000 C CNN
-F 2 "" H 10100 8200 50  0001 C CNN
-F 3 "" H 10100 8200 50  0001 C CNN
-	1    10100 8200
+P 9650 8200
+F 0 "#PWR018" H 9650 8050 50  0001 C CNN
+F 1 "+5V" H 9665 8373 50  0000 C CNN
+F 2 "" H 9650 8200 50  0001 C CNN
+F 3 "" H 9650 8200 50  0001 C CNN
+	1    9650 8200
 	1    0    0    -1
 $EndComp
@@
 L power:GND #PWR021
 U 1 1 5C188B1C
-P 10300 8700
-F 0 "#PWR021" H 10300 8450 50  0001 C CNN
-F 1 "GND" H 10305 8527 50  0000 C CNN
-F 2 "" H 10300 8700 50  0001 C CNN
-F 3 "" H 10300 8700 50  0001 C CNN
-	1    10300 8700
+P 10300 9000
+F 0 "#PWR021" H 10300 8750 50  0001 C CNN
+F 1 "GND" H 10305 8827 50  0000 C CNN
+F 2 "" H 10300 9000 50  0001 C CNN
+F 3 "" H 10300 9000 50  0001 C CNN
+	1    10300 9000
 	1    0    0    -1
 $EndComp
@@
 	1    0    0    -1
 $EndComp
-Wire Wire Line
-	10300 8200 10300 8300
-Wire Wire Line
-	10400 8300 10300 8300
 NoConn ~ 1650 1400
 NoConn ~ 1650 1500
@@
 NoConn ~ 3550 1500
 NoConn ~ 3550 1400
-$Comp
-L Regulator_Linear:MC78M05_TO252 U1
-U 1 1 5DB0F90A
-P 10300 6950
-F 0 "U1" H 10300 7192 50  0000 C CNN
-F 1 "MC78M05_TO252" H 10300 7101 50  0000 C CNN
-F 2 "Package_TO_SOT_SMD:TO-252-2" H 10300 7175 50  0001 C CIN
-F 3 "" H 10300 6900 50  0001 C CNN
-	1    10300 6950
-	1    0    0    -1
-$EndComp
 Wire Wire Line
 	10000 6950 9800 6950
-Wire Wire Line
-	9800 6950 9800 6750
 $Comp
 L power:+12V #PWR09
@@
 Wire Wire Line
 	10600 6950 10800 6950
-Wire Wire Line
-	10800 6950 10800 6750
 $Comp
 L power:+5V #PWR010
@@
 	1    10300 7500
 	1    0    0    -1
-$EndComp
-$Comp
-L Device:C C1
-U 1 1 5DB7525C
-P 9400 7200
-F 0 "C1" H 9285 7154 50  0000 R CNN
-F 1 "100n" H 9285 7245 50  0000 R CNN
-F 2 "Capacitor_SMD:C_0805_2012Metric" H 9438 7050 50  0001 C CNN
-F 3 "" H 9400 7200 50  0001 C CNN
-	1    9400 7200
-	1    0    0    1
 $EndComp
 $Comp
@@
 F 0 "C3" H 10915 7246 50  0000 L CNN
 F 1 "10u" H 10915 7155 50  0000 L CNN
-F 2 "Capacitor_SMD:C_1210_3225Metric_Pad1.42x2.65mm_HandSolder" H 10800 7200 50  0001 C CNN
+F 2 "Capacitor_Tantalum_SMD:CP_EIA-3528-15_AVX-H" H 10800 7200 50  0001 C CNN
 F 3 "" H 10800 7200 50  0001 C CNN
 	1    10800 7200
@@
 F 0 "J4" H 10679 8346 50  0000 L CNN
 F 1 "Screw_Terminal_01x04" H 10680 8301 50  0001 L CNN
-F 2 "Phoenix_MFKDS:Phoenix_MFKDS-5.08_1x04_P5.08mm" H 10600 8400 50  0001 C CNN
+F 2 "TerminalBlock:TerminalBlock_bornier-4_P5.08mm" H 10600 8400 50  0001 C CNN
 F 3 "" H 10600 8400 50  0001 C CNN
 	1    10600 8400
 	1    0    0    -1
 $EndComp
-Wire Wire Line
-	10100 8200 10100 8400
-Wire Wire Line
-	10100 8400 10400 8400
-Wire Wire Line
-	9900 8200 9900 8500
-Wire Wire Line
-	9900 8500 10400 8500
-Wire Wire Line
-	10300 8700 10300 8600
-Wire Wire Line
-	10300 8600 10400 8600
-Connection ~ 9800 7450
 Connection ~ 10800 7450
 Wire Wire Line
@@
 Wire Wire Line
 	11200 7450 11200 7350
-Wire Wire Line
-	9400 6950 9400 7050
-Wire Wire Line
-	9400 7350 9400 7450
 $Comp
 L Device:CP1 C2
@@
 F 0 "C2" H 9600 7250 50  0000 L CNN
 F 1 "10u" H 9550 7150 50  0000 L CNN
-F 2 "Capacitor_SMD:C_1210_3225Metric_Pad1.42x2.65mm_HandSolder" H 9800 7200 50  0001 C CNN
+F 2 "Capacitor_Tantalum_SMD:CP_EIA-3528-15_AVX-H" H 9800 7200 50  0001 C CNN
 F 3 "" H 9800 7200 50  0001 C CNN
 	1    9800 7200
 	1    0    0    -1
 $EndComp
-Wire Wire Line
-	9400 7450 9800 7450
-Wire Wire Line
-	9400 6950 9800 6950
 Wire Wire Line
 	10800 6950 11200 6950
@@
 Wire Wire Line
 	12250 1450 11750 1450
+Wire Wire Line
+	12250 1550 11750 1550
+Wire Wire Line
+	12250 1750 11750 1750
+Wire Wire Line
+	12250 1850 11750 1850
+Wire Wire Line
+	12250 2050 11750 2050
+Wire Wire Line
+	12250 2150 11750 2150
+Wire Wire Line
+	12250 2350 11750 2350
+Wire Wire Line
+	12250 2450 11750 2450
+Wire Wire Line
+	12250 2650 11750 2650
+Wire Wire Line
+	12250 2750 11750 2750
+Wire Wire Line
+	12250 2950 11750 2950
+Wire Wire Line
+	12250 3050 11750 3050
+Wire Wire Line
+	12250 3250 11750 3250
+Wire Wire Line
+	12250 3350 11750 3350
+Wire Wire Line
+	12250 3550 11750 3550
+Wire Wire Line
+	12250 3650 11750 3650
+Wire Wire Line
+	12250 3850 11750 3850
+Wire Wire Line
+	12250 3950 11750 3950
+Wire Wire Line
+	12250 4150 11750 4150
+Wire Wire Line
+	12250 4250 11750 4250
+Wire Wire Line
+	10800 6950 10800 6750
+Wire Wire Line
+	9800 6950 9800 6750
+$Comp
+L Regulator_Linear:MC78M05_TO252 U1
+U 1 1 5DB0F90A
+P 10300 6950
+F 0 "U1" H 10300 7192 50  0000 C CNN
+F 1 "MC78M05_TO252" H 10300 7101 50  0000 C CNN
+F 2 "Package_TO_SOT_SMD:TO-252-2" H 10300 7175 50  0001 C CIN
+F 3 "" H 10300 6900 50  0001 C CNN
+	1    10300 6950
+	1    0    0    -1
+$EndComp
+$Comp
+L power:GND #PWR0123
+U 1 1 5BA8843A
+P 10050 9000
+F 0 "#PWR0123" H 10050 8750 50  0001 C CNN
+F 1 "GND" H 10055 8827 50  0000 C CNN
+F 2 "" H 10050 9000 50  0001 C CNN
+F 3 "" H 10050 9000 50  0001 C CNN
+	1    10050 9000
+	1    0    0    -1
+$EndComp
+$Comp
+L Device:CP1 C19
+U 1 1 5BAD156E
+P 10050 8850
+F 0 "C19" H 9800 8900 50  0000 L CNN
+F 1 "10u" H 9800 8800 50  0000 L CNN
+F 2 "Capacitor_Tantalum_SMD:CP_EIA-3528-15_AVX-H" H 10050 8850 50  0001 C CNN
+F 3 "" H 10050 8850 50  0001 C CNN
+	1    10050 8850
+	1    0    0    -1
+$EndComp
+$Comp
+L Device:CP1 C18
+U 1 1 5BAD15CA
+P 9650 8850
+F 0 "C18" H 9400 8900 50  0000 L CNN
+F 1 "10u" H 9400 8800 50  0000 L CNN
+F 2 "Capacitor_Tantalum_SMD:CP_EIA-3528-15_AVX-H" H 9650 8850 50  0001 C CNN
+F 3 "" H 9650 8850 50  0001 C CNN
+	1    9650 8850
+	1    0    0    -1
+$EndComp
+$Comp
+L power:GND #PWR0125
+U 1 1 5BB0887E
+P 9650 9000
+F 0 "#PWR0125" H 9650 8750 50  0001 C CNN
+F 1 "GND" H 9655 8827 50  0000 C CNN
+F 2 "" H 9650 9000 50  0001 C CNN
+F 3 "" H 9650 9000 50  0001 C CNN
+	1    9650 9000
+	1    0    0    -1
+$EndComp
+$Comp
+L power:GND #PWR0124
+U 1 1 5BB088AB
+P 9250 9000
+F 0 "#PWR0124" H 9250 8750 50  0001 C CNN
+F 1 "GND" H 9255 8827 50  0000 C CNN
+F 2 "" H 9250 9000 50  0001 C CNN
+F 3 "" H 9250 9000 50  0001 C CNN
+	1    9250 9000
+	1    0    0    -1
+$EndComp
+$Comp
+L Device:CP1 C20
+U 1 1 5BB12861
+P 9250 8850
+F 0 "C20" H 9000 8900 50  0000 L CNN
+F 1 "10u" H 9000 8800 50  0000 L CNN
+F 2 "Capacitor_Tantalum_SMD:CP_EIA-3528-15_AVX-H" H 9250 8850 50  0001 C CNN
+F 3 "" H 9250 8850 50  0001 C CNN
+	1    9250 8850
+	1    0    0    -1
+$EndComp
+$Comp
+L Mechanical:MountingHole MH1
+U 1 1 5BB1C4CD
+P 12950 8050
+F 0 "MH1" H 13050 8096 50  0000 L CNN
+F 1 "MountingHole" H 13050 8005 50  0000 L CNN
+F 2 "HSMC:MountingHole" H 12950 8050 50  0001 C CNN
+F 3 "~" H 12950 8050 50  0001 C CNN
+	1    12950 8050
+	1    0    0    -1
+$EndComp
+$Comp
+L Mechanical:MountingHole MH2
+U 1 1 5BB1C6A7
+P 12950 8300
+F 0 "MH2" H 13050 8346 50  0000 L CNN
+F 1 "MountingHole" H 13050 8255 50  0000 L CNN
+F 2 "HSMC:MountingHole" H 12950 8300 50  0001 C CNN
+F 3 "~" H 12950 8300 50  0001 C CNN
+	1    12950 8300
+	1    0    0    -1
+$EndComp
+Wire Wire Line
+	10300 8300 10400 8300
+Wire Wire Line
+	10300 8300 10300 9000
+Wire Wire Line
+	9250 8200 9250 8600
+Wire Wire Line
+	9650 8200 9650 8500
+Wire Wire Line
+	10050 8200 10050 8400
+Wire Wire Line
+	10400 8400 10050 8400
+Connection ~ 10050 8400
+Wire Wire Line
+	10050 8400 10050 8700
+Wire Wire Line
+	10400 8500 9650 8500
+Connection ~ 9650 8500
+Wire Wire Line
+	9650 8500 9650 8700
+Wire Wire Line
+	10400 8600 9250 8600
 Wire Bus Line
 	8300 900  13050 900
 Wire Bus Line
+	8200 1000 8200 4100
+Wire Bus Line
 	12350 1000 12350 4150
-Wire Bus Line
-	8200 1000 8200 4100
-Wire Wire Line
-	12250 1550 11750 1550
-Wire Wire Line
-	12250 1750 11750 1750
-Wire Wire Line
-	12250 1850 11750 1850
-Wire Wire Line
-	12250 2050 11750 2050
-Wire Wire Line
-	12250 2150 11750 2150
-Wire Wire Line
-	12250 2350 11750 2350
-Wire Wire Line
-	12250 2450 11750 2450
-Wire Wire Line
-	12250 2650 11750 2650
-Wire Wire Line
-	12250 2750 11750 2750
-Wire Wire Line
-	12250 2950 11750 2950
-Wire Wire Line
-	12250 3050 11750 3050
-Wire Wire Line
-	12250 3250 11750 3250
-Wire Wire Line
-	12250 3350 11750 3350
-Wire Wire Line
-	12250 3550 11750 3550
-Wire Wire Line
-	12250 3650 11750 3650
-Wire Wire Line
-	12250 3850 11750 3850
-Wire Wire Line
-	12250 3950 11750 3950
-Wire Wire Line
-	12250 4150 11750 4150
-Wire Wire Line
-	12250 4250 11750 4250
+Connection ~ 9250 8600
+Wire Wire Line
+	9250 8600 9250 8700
 $EndSCHEMATC

Commit message: Reroute GPIO pins (again)
Changed lines of the file:
@@
 	11850 4350 11750 4350
-Wire Wire Line
-	11850 4050 11750 4050
 Wire Wire Line
 	9750 4350 9850 4350
@@
 Entry Bus Bus
 	8200 1000 8300 900
-Text Label 8050 1400 2    50   ~ 0
-GPIO0
-Text Label 8050 1500 2    50   ~ 0
-GPIO1
-Text Label 8050 1700 2    50   ~ 0
-GPIO2
-Text Label 8050 1800 2    50   ~ 0
-GPIO3
-Text Label 8050 2000 2    50   ~ 0
-GPIO4
-Text Label 8050 2100 2    50   ~ 0
-GPIO5
-Text Label 8050 2300 2    50   ~ 0
-GPIO6
-Text Label 8050 2400 2    50   ~ 0
-GPIO7
-Text Label 8050 2600 2    50   ~ 0
-GPIO8
-Text Label 8050 2700 2    50   ~ 0
-GPIO9
-Text Label 8050 2900 2    50   ~ 0
-GPIO10
-Text Label 8050 3000 2    50   ~ 0
-GPIO11
-Text Label 8050 3200 2    50   ~ 0
-GPIO12
-Text Label 8050 3300 2    50   ~ 0
-GPIO13
-Text Label 8050 3500 2    50   ~ 0
-GPIO14
-Text Label 8050 3600 2    50   ~ 0
-GPIO15
-Text Label 8050 3800 2    50   ~ 0
-GPIO16
-Text Label 8050 3900 2    50   ~ 0
-GPIO17
-Text Label 8050 4100 2    50   ~ 0
-GPIO18
-Text Label 8050 4200 2    50   ~ 0
-GPIO19
-Wire Wire Line
-	7600 1400 8100 1400
-Wire Wire Line
-	7600 1500 8100 1500
-Wire Wire Line
-	7600 1700 8100 1700
-Wire Wire Line
-	7600 1800 8100 1800
-Wire Wire Line
-	7600 2000 8100 2000
-Wire Wire Line
-	7600 2100 8100 2100
-Wire Wire Line
-	7600 2300 8100 2300
-Wire Wire Line
-	7600 2400 8100 2400
-Wire Wire Line
-	7600 2600 8100 2600
-Wire Wire Line
-	7600 2700 8100 2700
-Wire Wire Line
-	7600 2900 8100 2900
-Wire Wire Line
-	7600 3000 8100 3000
-Wire Wire Line
-	7600 3200 8100 3200
-Wire Wire Line
-	7600 3300 8100 3300
-Wire Wire Line
-	7600 3500 8100 3500
-Wire Wire Line
-	7600 3600 8100 3600
-Wire Wire Line
-	7600 3800 8100 3800
-Wire Wire Line
-	7600 3900 8100 3900
-Wire Wire Line
-	7600 4100 8100 4100
-Wire Wire Line
-	7600 4200 8100 4200
-Text Label 12200 1450 2    50   ~ 0
-GPIO20
-Text Label 12200 1550 2    50   ~ 0
-GPIO21
-Text Label 12200 1750 2    50   ~ 0
-GPIO22
-Text Label 12200 1850 2    50   ~ 0
-GPIO23
-Text Label 12200 2050 2    50   ~ 0
-GPIO24
-Text Label 12200 2150 2    50   ~ 0
-GPIO25
-Text Label 12200 2350 2    50   ~ 0
-GPIO26
-Text Label 12200 2450 2    50   ~ 0
-GPIO27
-Text Label 12200 2650 2    50   ~ 0
-GPIO28
-Text Label 12200 2750 2    50   ~ 0
-GPIO29
-Text Label 12200 2950 2    50   ~ 0
-GPIO30
-Text Label 12200 3050 2    50   ~ 0
-GPIO31
-Text Label 12200 3250 2    50   ~ 0
-GPIO32
-Text Label 12200 3350 2    50   ~ 0
-GPIO33
-Text Label 12200 3550 2    50   ~ 0
-GPIO34
-Text Label 12200 3650 2    50   ~ 0
-GPIO35
-Text Label 12200 3850 2    50   ~ 0
-GPIO36
-Text Label 12200 3950 2    50   ~ 0
-GPIO37
-Text Label 12200 4150 2    50   ~ 0
-GPIO38
-Text Label 12200 4250 2    50   ~ 0
-GPIO39
-Wire Wire Line
-	12250 1450 11750 1450
-Wire Wire Line
-	12250 1550 11750 1550
-Wire Wire Line
-	12250 1750 11750 1750
-Wire Wire Line
-	12250 1850 11750 1850
-Wire Wire Line
-	12250 2050 11750 2050
-Wire Wire Line
-	12250 2150 11750 2150
-Wire Wire Line
-	12250 2350 11750 2350
-Wire Wire Line
-	12250 2450 11750 2450
-Wire Wire Line
-	12250 2650 11750 2650
-Wire Wire Line
-	12250 2750 11750 2750
-Wire Wire Line
-	12250 2950 11750 2950
-Wire Wire Line
-	12250 3050 11750 3050
-Wire Wire Line
-	12250 3250 11750 3250
-Wire Wire Line
-	12250 3350 11750 3350
-Wire Wire Line
-	12250 3550 11750 3550
-Wire Wire Line
-	12250 3650 11750 3650
-Wire Wire Line
-	12250 3850 11750 3850
-Wire Wire Line
-	12250 3950 11750 3950
-Wire Wire Line
-	12250 4150 11750 4150
-Wire Wire Line
-	12250 4250 11750 4250
 Wire Wire Line
 	10800 6950 10800 6750
@@
 Wire Wire Line
 	10400 8600 9250 8600
+Connection ~ 9250 8600
+Wire Wire Line
+	9250 8600 9250 8700
+Text Label 8050 1400 2    50   ~ 0
+GPIO39
+Text Label 8050 1500 2    50   ~ 0
+GPIO38
+Text Label 8050 1700 2    50   ~ 0
+GPIO37
+Text Label 8050 1800 2    50   ~ 0
+GPIO36
+Text Label 8050 2000 2    50   ~ 0
+GPIO35
+Text Label 8050 2100 2    50   ~ 0
+GPIO34
+Text Label 8050 2300 2    50   ~ 0
+GPIO33
+Text Label 8050 2400 2    50   ~ 0
+GPIO32
+Text Label 8050 2600 2    50   ~ 0
+GPIO31
+Text Label 8050 2700 2    50   ~ 0
+GPIO30
+Text Label 8050 2900 2    50   ~ 0
+GPIO29
+Text Label 8050 3000 2    50   ~ 0
+GPIO28
+Text Label 8050 3200 2    50   ~ 0
+GPIO27
+Text Label 8050 3300 2    50   ~ 0
+GPIO26
+Text Label 8050 3500 2    50   ~ 0
+GPIO25
+Text Label 8050 3600 2    50   ~ 0
+GPIO24
+Text Label 8050 3800 2    50   ~ 0
+GPIO23
+Text Label 8050 3900 2    50   ~ 0
+GPIO22
+Text Label 8050 4100 2    50   ~ 0
+GPIO21
+Text Label 8050 4200 2    50   ~ 0
+GPIO20
+Text Label 12200 1450 2    50   ~ 0
+GPIO19
+Text Label 12200 1550 2    50   ~ 0
+GPIO18
+Text Label 12200 1750 2    50   ~ 0
+GPIO17
+Text Label 12200 1850 2    50   ~ 0
+GPIO16
+Text Label 12200 2050 2    50   ~ 0
+GPIO15
+Text Label 12200 2150 2    50   ~ 0
+GPIO14
+Text Label 12200 2350 2    50   ~ 0
+GPIO13
+Text Label 12200 2450 2    50   ~ 0
+GPIO12
+Text Label 12200 2650 2    50   ~ 0
+GPIO11
+Text Label 12200 2750 2    50   ~ 0
+GPIO10
+Text Label 12200 2950 2    50   ~ 0
+GPIO9
+Text Label 12200 3050 2    50   ~ 0
+GPIO8
+Text Label 12200 3250 2    50   ~ 0
+GPIO7
+Text Label 12200 3350 2    50   ~ 0
+GPIO6
+Text Label 12200 3550 2    50   ~ 0
+GPIO5
+Text Label 12200 3650 2    50   ~ 0
+GPIO4
+Text Label 12200 3850 2    50   ~ 0
+GPIO3
+Text Label 12200 3950 2    50   ~ 0
+GPIO2
+Text Label 12200 4150 2    50   ~ 0
+GPIO1
+Text Label 12200 4250 2    50   ~ 0
+GPIO0
+Wire Wire Line
+	12250 1450 11750 1450
+Wire Wire Line
+	12250 1550 11750 1550
+Wire Wire Line
+	12250 1750 11750 1750
+Wire Wire Line
+	12250 1850 11750 1850
+Wire Wire Line
+	12250 2050 11750 2050
+Wire Wire Line
+	12250 2150 11750 2150
+Wire Wire Line
+	12250 2350 11750 2350
+Wire Wire Line
+	12250 2450 11750 2450
+Wire Wire Line
+	12250 2650 11750 2650
+Wire Wire Line
+	12250 2750 11750 2750
+Wire Wire Line
+	12250 2950 11750 2950
+Wire Wire Line
+	12250 3050 11750 3050
+Wire Wire Line
+	12250 3250 11750 3250
+Wire Wire Line
+	12250 3350 11750 3350
+Wire Wire Line
+	12250 3550 11750 3550
+Wire Wire Line
+	12250 3650 11750 3650
+Wire Wire Line
+	12250 3850 11750 3850
+Wire Wire Line
+	12250 3950 11750 3950
+Wire Wire Line
+	12250 4150 11750 4150
+Wire Wire Line
+	12250 4250 11750 4250
+Wire Wire Line
+	7600 1400 8100 1400
+Wire Wire Line
+	7600 1500 8100 1500
+Wire Wire Line
+	7600 1700 8100 1700
+Wire Wire Line
+	7600 1800 8100 1800
+Wire Wire Line
+	7600 2000 8100 2000
+Wire Wire Line
+	7600 2100 8100 2100
+Wire Wire Line
+	7600 2300 8100 2300
+Wire Wire Line
+	7600 2400 8100 2400
+Wire Wire Line
+	7600 2600 8100 2600
+Wire Wire Line
+	7600 2700 8100 2700
+Wire Wire Line
+	7600 2900 8100 2900
+Wire Wire Line
+	7600 3000 8100 3000
+Wire Wire Line
+	7600 3200 8100 3200
+Wire Wire Line
+	7600 3300 8100 3300
+Wire Wire Line
+	7600 3500 8100 3500
+Wire Wire Line
+	7600 3600 8100 3600
+Wire Wire Line
+	7600 3800 8100 3800
+Wire Wire Line
+	7600 3900 8100 3900
+Wire Wire Line
+	7600 4100 8100 4100
+Wire Wire Line
+	7600 4200 8100 4200
+Wire Wire Line
+	11850 4050 11750 4050
 Wire Bus Line
 	8300 900  13050 900
 Wire Bus Line
+	12350 1000 12350 4150
+Wire Bus Line
 	8200 1000 8200 4100
-Wire Bus Line
-	12350 1000 12350 4150
-Connection ~ 9250 8600
-Wire Wire Line
-	9250 8600 9250 8700
 $EndSCHEMATC
