File: HSMC-GPIO-kicad.sch (KiCad schematic (older format))
At the start: 16 parts, among them J1 HSMC, J2 Conn_01x03_Male, J3 I2C, J4 Screw_Terminal_01x04, U1 MC78M05_TO252, U2 TCA9517

Commit message: Fix issues and reroute I2C buffer, length match GPIO bus
Parts:
- removed U2: TCA9517, Package_SO:SOIC-8_3.9x4.9mm_P1.27mm, symbol TCA9517:TCA9517
- added R41, R42: 10k, Resistor_SMD:R_0603_1608Metric, symbol Device:R
- added R43, R44: 2k, Resistor_SMD:R_0603_1608Metric, symbol Device:R
- added U2: PCA9507, Package_SO:SOIC-8_3.9x4.9mm_P1.27mm, symbol PCA95xx:PCA9507
- C18, C19, C2, C20, C3: footprint Capacitor_Tantalum_SMD:CP_EIA-3528-15_AVX-H -> Capacitor_Tantalum_SMD:CP_EIA-3528-21_Kemet-B
Connections:
- net labels added: VBUS
- net labels removed: VI2C
- wire segments 193 -> 210
Other:
- moved on the sheet: C5, C6

Commit message: Rotate GPIO connector 180deg, reroute
Changed lines of the file:
@@
 Wire Wire Line
 	10300 8300 10300 9000
-Text Label 8050 1400 2    50   ~ 0
-GPIO39
-Text Label 8050 1500 2    50   ~ 0
-GPIO38
-Text Label 8050 1700 2    50   ~ 0
-GPIO37
-Text Label 8050 1800 2    50   ~ 0
-GPIO36
-Text Label 8050 2000 2    50   ~ 0
-GPIO35
-Text Label 8050 2100 2    50   ~ 0
-GPIO34
-Text Label 8050 2300 2    50   ~ 0
-GPIO33
-Text Label 8050 2400 2    50   ~ 0
-GPIO32
-Text Label 8050 2600 2    50   ~ 0
-GPIO31
-Text Label 8050 2700 2    50   ~ 0
-GPIO30
-Text Label 8050 2900 2    50   ~ 0
-GPIO29
-Text Label 8050 3000 2    50   ~ 0
-GPIO28
-Text Label 8050 3200 2    50   ~ 0
-GPIO27
-Text Label 8050 3300 2    50   ~ 0
-GPIO26
-Text Label 8050 3500 2    50   ~ 0
-GPIO25
-Text Label 8050 3600 2    50   ~ 0
-GPIO24
-Text Label 8050 3800 2    50   ~ 0
-GPIO23
-Text Label 8050 3900 2    50   ~ 0
-GPIO22
-Text Label 8050 4100 2    50   ~ 0
-GPIO21
-Text Label 8050 4200 2    50   ~ 0
-GPIO20
-Text Label 12200 1450 2    50   ~ 0
-GPIO19
-Text Label 12200 1550 2    50   ~ 0
-GPIO18
-Text Label 12200 1750 2    50   ~ 0
-GPIO17
-Text Label 12200 1850 2    50   ~ 0
-GPIO16
-Text Label 12200 2050 2    50   ~ 0
-GPIO15
-Text Label 12200 2150 2    50   ~ 0
-GPIO14
-Text Label 12200 2350 2    50   ~ 0
-GPIO13
-Text Label 12200 2450 2    50   ~ 0
-GPIO12
-Text Label 12200 2650 2    50   ~ 0
-GPIO11
-Text Label 12200 2750 2    50   ~ 0
-GPIO10
-Text Label 12200 2950 2    50   ~ 0
-GPIO9
-Text Label 12200 3050 2    50   ~ 0
-GPIO8
-Text Label 12200 3250 2    50   ~ 0
-GPIO7
-Text Label 12200 3350 2    50   ~ 0
-GPIO6
-Text Label 12200 3550 2    50   ~ 0
-GPIO5
-Text Label 12200 3650 2    50   ~ 0
-GPIO4
-Text Label 12200 3850 2    50   ~ 0
-GPIO3
-Text Label 12200 3950 2    50   ~ 0
-GPIO2
-Text Label 12200 4150 2    50   ~ 0
-GPIO1
-Text Label 12200 4250 2    50   ~ 0
-GPIO0
-Wire Wire Line
-	12250 1450 11750 1450
-Wire Wire Line
-	12250 1550 11750 1550
-Wire Wire Line
-	12250 1750 11750 1750
-Wire Wire Line
-	12250 1850 11750 1850
-Wire Wire Line
-	12250 2050 11750 2050
-Wire Wire Line
-	12250 2150 11750 2150
-Wire Wire Line
-	12250 2350 11750 2350
-Wire Wire Line
-	12250 2450 11750 2450
-Wire Wire Line
-	12250 2650 11750 2650
-Wire Wire Line
-	12250 2750 11750 2750
-Wire Wire Line
-	12250 2950 11750 2950
-Wire Wire Line
-	12250 3050 11750 3050
-Wire Wire Line
-	12250 3250 11750 3250
-Wire Wire Line
-	12250 3350 11750 3350
-Wire Wire Line
-	12250 3550 11750 3550
-Wire Wire Line
-	12250 3650 11750 3650
-Wire Wire Line
-	12250 3850 11750 3850
-Wire Wire Line
-	12250 3950 11750 3950
-Wire Wire Line
-	12250 4150 11750 4150
-Wire Wire Line
-	12250 4250 11750 4250
-Wire Wire Line
-	7600 1400 8100 1400
-Wire Wire Line
-	7600 1500 8100 1500
-Wire Wire Line
-	7600 1700 8100 1700
-Wire Wire Line
-	7600 1800 8100 1800
-Wire Wire Line
-	7600 2000 8100 2000
-Wire Wire Line
-	7600 2100 8100 2100
-Wire Wire Line
-	7600 2300 8100 2300
-Wire Wire Line
-	7600 2400 8100 2400
-Wire Wire Line
-	7600 2600 8100 2600
-Wire Wire Line
-	7600 2700 8100 2700
-Wire Wire Line
-	7600 2900 8100 2900
-Wire Wire Line
-	7600 3000 8100 3000
-Wire Wire Line
-	7600 3200 8100 3200
-Wire Wire Line
-	7600 3300 8100 3300
-Wire Wire Line
-	7600 3500 8100 3500
-Wire Wire Line
-	7600 3600 8100 3600
-Wire Wire Line
-	7600 3800 8100 3800
-Wire Wire Line
-	7600 3900 8100 3900
-Wire Wire Line
-	7600 4100 8100 4100
-Wire Wire Line
-	7600 4200 8100 4200
 Wire Wire Line
 	11850 4050 11750 4050
@@
 Wire Wire Line
 	7250 8300 7250 8400
+Wire Wire Line
+	7250 8400 7700 8400
+Text Label 8050 1400 2    50   ~ 0
+GPIO0
+Text Label 8050 1500 2    50   ~ 0
+GPIO1
+Text Label 8050 1700 2    50   ~ 0
+GPIO2
+Text Label 8050 1800 2    50   ~ 0
+GPIO3
+Text Label 8050 2000 2    50   ~ 0
+GPIO4
+Text Label 8050 2100 2    50   ~ 0
+GPIO5
+Text Label 8050 2300 2    50   ~ 0
+GPIO6
+Text Label 8050 2400 2    50   ~ 0
+GPIO7
+Text Label 8050 2600 2    50   ~ 0
+GPIO8
+Text Label 8050 2700 2    50   ~ 0
+GPIO9
+Text Label 8050 2900 2    50   ~ 0
+GPIO10
+Text Label 8050 3000 2    50   ~ 0
+GPIO11
+Text Label 8050 3200 2    50   ~ 0
+GPIO12
+Text Label 8050 3300 2    50   ~ 0
+GPIO13
+Text Label 8050 3500 2    50   ~ 0
+GPIO14
+Text Label 8050 3600 2    50   ~ 0
+GPIO15
+Text Label 8050 3800 2    50   ~ 0
+GPIO16
+Text Label 8050 3900 2    50   ~ 0
+GPIO17
+Text Label 8050 4100 2    50   ~ 0
+GPIO18
+Text Label 8050 4200 2    50   ~ 0
+GPIO19
+Text Label 12200 1450 2    50   ~ 0
+GPIO20
+Text Label 12200 1550 2    50   ~ 0
+GPIO21
+Text Label 12200 1750 2    50   ~ 0
+GPIO22
+Text Label 12200 1850 2    50   ~ 0
+GPIO23
+Text Label 12200 2050 2    50   ~ 0
+GPIO24
+Text Label 12200 2150 2    50   ~ 0
+GPIO25
+Text Label 12200 2350 2    50   ~ 0
+GPIO26
+Text Label 12200 2450 2    50   ~ 0
+GPIO27
+Text Label 12200 2650 2    50   ~ 0
+GPIO28
+Text Label 12200 2750 2    50   ~ 0
+GPIO29
+Text Label 12200 2950 2    50   ~ 0
+GPIO30
+Text Label 12200 3050 2    50   ~ 0
+GPIO31
+Text Label 12200 3250 2    50   ~ 0
+GPIO32
+Text Label 12200 3350 2    50   ~ 0
+GPIO33
+Text Label 12200 3550 2    50   ~ 0
+GPIO34
+Text Label 12200 3650 2    50   ~ 0
+GPIO35
+Text Label 12200 3850 2    50   ~ 0
+GPIO36
+Text Label 12200 3950 2    50   ~ 0
+GPIO37
+Text Label 12200 4150 2    50   ~ 0
+GPIO38
+Text Label 12200 4250 2    50   ~ 0
+GPIO39
+Wire Wire Line
+	8100 1400 7600 1400
+Wire Wire Line
+	8100 1500 7600 1500
+Wire Wire Line
+	8100 1700 7600 1700
+Wire Wire Line
+	8100 1800 7600 1800
+Wire Wire Line
+	8100 2000 7600 2000
+Wire Wire Line
+	8100 2100 7600 2100
+Wire Wire Line
+	8100 2300 7600 2300
+Wire Wire Line
+	8100 2400 7600 2400
+Wire Wire Line
+	8100 2600 7600 2600
+Wire Wire Line
+	8100 2700 7600 2700
+Wire Wire Line
+	8100 2900 7600 2900
+Wire Wire Line
+	8100 3000 7600 3000
+Wire Wire Line
+	8100 3200 7600 3200
+Wire Wire Line
+	8100 3300 7600 3300
+Wire Wire Line
+	8100 3500 7600 3500
+Wire Wire Line
+	8100 3600 7600 3600
+Wire Wire Line
+	8100 3800 7600 3800
+Wire Wire Line
+	8100 3900 7600 3900
+Wire Wire Line
+	8100 4100 7600 4100
+Wire Wire Line
+	8100 4200 7600 4200
+Wire Wire Line
+	11750 1450 12250 1450
+Wire Wire Line
+	11750 1550 12250 1550
+Wire Wire Line
+	11750 1750 12250 1750
+Wire Wire Line
+	11750 1850 12250 1850
+Wire Wire Line
+	11750 2050 12250 2050
+Wire Wire Line
+	11750 2150 12250 2150
+Wire Wire Line
+	11750 2350 12250 2350
+Wire Wire Line
+	11750 2450 12250 2450
+Wire Wire Line
+	11750 2650 12250 2650
+Wire Wire Line
+	11750 2750 12250 2750
+Wire Wire Line
+	11750 2950 12250 2950
+Wire Wire Line
+	11750 3050 12250 3050
+Wire Wire Line
+	11750 3250 12250 3250
+Wire Wire Line
+	11750 3350 12250 3350
+Wire Wire Line
+	11750 3550 12250 3550
+Wire Wire Line
+	11750 3650 12250 3650
+Wire Wire Line
+	11750 3850 12250 3850
+Wire Wire Line
+	11750 3950 12250 3950
+Wire Wire Line
+	11750 4150 12250 4150
+Wire Wire Line
+	11750 4250 12250 4250
 Wire Bus Line
-	8300 900  13050 900
+	12350 1000 12350 4150
 Wire Bus Line
 	8200 1000 8200 4100
 Wire Bus Line
-	12350 1000 12350 4150
-Wire Wire Line
-	7250 8400 7700 8400
+	8300 900  13050 900
 $EndSCHEMATC

Commit message: Modify and submit to Sunstone for DFM report.
Parts:
- removed J1: HSMC, HSMC:HSMC_Card_QTH-090-01-L-D-A, symbol HSMC:HSMC
- removed J2: Conn_01x03_Male, Connector_PinHeader_2.54mm:PinHeader_1x03_P2.54mm_Vertical, symbol Connector:Conn_01x03_Male
- removed MH1, MH2: MountingHole, HSMC:MountingHole, symbol Mechanical:MountingHole
- added D41, D42: BAT54S, Package_TO_SOT_SMD:SOT-23, symbol Diode:BAT54S
- added J1: HSMC_Card_QTH, Connector_Samtec:Samtec_HSMC_Card_QTH-090-01-x-D-A_3.076x0.932in_P0.5mm_Vertical, symbol Connector:HSMC_Card_QTH
- added JP1: Jumper_3_Bridged12, Connector_PinHeader_2.54mm:PinHeader_1x03_P2.54mm_Vertical, symbol Jumper:Jumper_3_Bridged12
- U2: symbol PCA95xx:PCA9507 -> Interface:PCA9507
Connections:
- wire segments 210 -> 229
Other:
- moved on the sheet: R41, R42, R43, R44

Commit message: Reroute GPIO, 5V regulator, and I2C buffer
Parts:
- removed C4: 100n, Capacitor_SMD:C_0805_2012Metric, symbol Device:C
- added LOGO1: Logo_Open_Hardware_Small, Symbol:OSHW-Logo2_7.3x6mm_Copper, symbol Graphic:Logo_Open_Hardware_Small
- renumbered C5 to C14, C6 to C15, C2 to C16, C3 to C17, C20 to C18, C18 to C19, C19 to C20, J1 to J2
Connections:
- wire segments 229 -> 225

Commit message: Minor footprint and position adjustments
Parts:
- LOGO1: footprint Symbol:OSHW-Logo2_7.3x6mm_Copper -> Symbol:OSHW-Symbol_6.7x6mm_SilkScreen
Changed lines of the file:
@@
 F 0 "LOGO1" H 12600 9875 50  0001 C CNN
 F 1 "Logo_Open_Hardware_Small" H 12600 9375 50  0001 C CNN
-F 2 "Symbol:OSHW-Logo2_7.3x6mm_Copper" H 12600 9600 50  0001 C CNN
+F 2 "Symbol:OSHW-Symbol_6.7x6mm_SilkScreen" H 12600 9600 50  0001 C CNN
 F 3 "~" H 12600 9600 50  0001 C CNN
 	1    12600 9600

Commit message: Updated to use new KLC-compliant symbols and footprints
Parts:
- removed J2: HSMC_Card_QTH, Connector_Samtec:Samtec_HSMC_Card_QTH-090-01-x-D-A_3.076x0.932in_P0.5mm_Vertical, symbol Connector:HSMC_Card_QTH
- removed U2: PCA9507, Package_SO:SOIC-8_3.9x4.9mm_P1.27mm, symbol Interface:PCA9507
- added J2: HSMC_Card_QTH, Connector_Samtec:Samtec_HSMC_Card_QTH-090-01-x-D-A_3.076x0.932in_P0.5mm_Vertical, symbol HSMC-GPIO-kicad-rescue:HSMC_Card_QTH-Connector_HSMC
- added U2: PCA9507, Package_SO:SOIC-8_3.9x4.9mm_P1.27mm, symbol PCA95xx:PCA9507
Connections:
- wire segments 225 -> 145
